File: hardware/cpu.kicad_sch (KiCad schematic)
At the start: 62 parts, among them Q5 MMBT3904, U1 H3, Y1 32kHz, Y3 24MHz

Commit message: Finished with V1!
Connections:
- net BT_WAKE: now also U1.D6 (PA2); no longer U1.D5 (PA1)
- net STATUS_LED: now also U1.C14 (PA17)
- net GPIO7: now reaches U1.A13 (PA20)
- net GPIO11: now reaches U1.A14 (PA21)
- net GPIO3: now reaches U1.B12 (PE12)
- net GPIO12: now reaches U1.B13 (PA18)
- net GPIO13: now reaches U1.B14 (PA19)
- net GPIO5: now reaches U1.C12 (PE9)
- net GPIO16: now reaches U1.C13 (PA12)
- net GPIO8: now reaches U1.D11 (PA0)
- net GPIO21: now reaches U1.D15 (PA16)
- net GPIO15: now reaches U1.E14 (PA6)
- net GPIO24: now reaches U1.E15 (PA13)
- net GPIO19: now reaches U1.F14 (PA15)
- net GPIO23: now reaches U1.G12 (PA14)
- new net GPIO10: U1.D5 (PA1)
