File: hardware/gpio.kicad_sch (KiCad schematic)
At the start: 10 parts, among them J8 Conn_01x03, J9 GPIO, Q4 BSN20

Commit message: Finished with V1!
Parts:
- D3, D4: footprint (none) -> LED_SMD:LED_0603_1608Metric; LCSC Part # (none) -> C965804
- J8: value Conn_01x03 -> UART
- J9: now not fitted
Connections:
- net GPIO10: now reaches J9.10 (Pin_10)
- net GPIO11: now reaches J9.11 (Pin_11)
- net GPIO12: now reaches J9.12 (Pin_12)
- net GPIO13: now reaches J9.13 (Pin_13)
- net GPIO15: now reaches J9.15 (Pin_15)
- net GPIO16: now reaches J9.16 (Pin_16)
- net GPIO17: now reaches J9.17 (Pin_17)
- net GPIO18: now reaches J9.18 (Pin_18)
- net GPIO19: now reaches J9.19 (Pin_19)
- net GPIO21: now reaches J9.21 (Pin_21)
- net GPIO22: now reaches J9.22 (Pin_22)
- net GPIO23: now reaches J9.23 (Pin_23)
- net GPIO24: now reaches J9.24 (Pin_24)
- net GPIO26: now reaches J9.26 (Pin_26)
- net GPIO27: now reaches J9.27 (Pin_27)
- net GPIO28: now reaches J9.28 (Pin_28)
- net GPIO29: now reaches J9.29 (Pin_29)
- net GPIO3: now reaches J9.3 (Pin_3)
- net GPIO31: now reaches J9.31 (Pin_31)
- net GPIO32: now reaches J9.32 (Pin_32)
- net GPIO33: now reaches J9.33 (Pin_33)
- net GPIO35: now reaches J9.35 (Pin_35)
- net GPIO36: now reaches J9.36 (Pin_36)
- net GPIO37: now reaches J9.37 (Pin_37)
- net GPIO38: now reaches J9.38 (Pin_38)
- net GPIO40: now reaches J9.40 (Pin_40)
- net GPIO5: now reaches J9.5 (Pin_5)
- net GPIO7: now reaches J9.7 (Pin_7)
- net GPIO8: now reaches J9.8 (Pin_8)
Other:
- note removed: "TODO: LED"
- moved on the sheet: D3, D4, J8, Q4, R56, R57, R58, R71, R72
