File: hardware/gpio.kicad_sch (KiCad schematic)
At the start: 10 parts, among them J8 UART, J9 GPIO, Q4 BSN20

Commit message: Add fixes and improvements
Parts:
- R71, R72: value 2.2k -> 2k; LCSC Part # C25879 -> C4109
Other:
- note removed: "TVS omitted because well I'm on a budget..."
Changed lines of the file:
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@@
 	(title_block
 		(title "Icepi CM0")
-		(date "2025-11-15")
+		(date "2025-11-21")
 		(rev "v1.0")
 		(company "Icy Electronics")
 		(comment 1 "Chengyin Yao (cheyao)")
 		(comment 2 "https://github.com/cheyao/icepi-cm0")
+		(comment 3 "License: Solderpad")
 	)
 	(bus_alias "CPU_UART"
@@
 	(bus_alias "GPIO"
 		(members "GPIO[0..40]")
-	)
-	(text "TVS omitted because well\nI'm on a budget..."
-		(exclude_from_sim no)
-		(at 195.834 120.396 0)
-		(effects
-			(font
-				(size 1.27 1.27)
-			)
-		)
 	)
 	(junction
@@
 			)
 		)
-		(property "Value" "2.2k"
+		(property "Value" "2k"
 			(at 176.53 81.28 90)
 			(effects
@@
 			)
 		)
-		(property "LCSC Part #" "C25879"
+		(property "LCSC Part #" "C4109"
 			(at 177.8 88.9 0)
 			(effects
@@
 			)
 		)
-		(property "Value" "2.2k"
+		(property "Value" "2k"
 			(at 176.53 69.85 90)
 			(effects
@@
 			)
 		)
-		(property "LCSC Part #" "C25879"
+		(property "LCSC Part #" "C4109"
 			(at 177.8 77.47 0)
 			(effects
