File: hardware/storage.kicad_sch (KiCad schematic)
At the start: 9 parts, among them J6 Micro_SD_Card_Det1, U21 EMMC5.1_BGA153

Commit message: Finished with V1!
Parts:
- U21: LCSC Part # (none) -> C5821038
