File: hardware/storage.kicad_sch (KiCad schematic)
At the start: 9 parts, among them J6 Micro_SD_Card_Det1, U21 EMMC5.1_BGA153

Commit message: Add fixes and improvements
Parts:
- added C133, C137: 4.7uF, Capacitor_SMD:C_0402_1005Metric, symbol Device:C
- added C134, C136: 100nF, Capacitor_SMD:C_0402_1005Metric, symbol Device:C
- added C135: 1uF, Capacitor_SMD:C_0402_1005Metric, symbol Device:C
Connections:
- net +3V3_IO: now also C133.1, C134.2, C135.2, C136.2, C137.1
- net GND: now also C133.2, C134.1, C135.1, C136.1, C137.2
Other:
- note added: "VCC"
- note added: "VCCQ"
