File: hardware/wifi.kicad_sch (KiCad schematic)
At the start: 33 parts, among them J11 ANT, J7 RJ45_Hanrun_HR913550A_Horizon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, U22 AP6212, U24 AW13412HDNR, Y2 26MHz

Commit message: Finished with V1!
Parts:
- C6: footprint (none) -> Capacitor_SMD:C_0402_1005Metric
- C74: LCSC Part # (none) -> C1523
- C9: LCSC Part # (none) -> C1546
