File: hardware/cm0.kicad_sch (KiCad schematic)
At the start: 0 parts

Commit message: Finished with V1!
Other:
- sheet GPIO ports: added {GPIO}; removed none
- sheet H3 ports: added {GPIO}; removed none
