File: hardware/ddr3.kicad_sch (KiCad schematic)
At the start: 22 parts, among them U2 H5TQ4G63EFR

Commit message: Add fixes and improvements
Parts:
- added C132: 100nF, Capacitor_SMD:C_0402_1005Metric, symbol Device:C
- R7, R8: value 2.2k -> 2k; LCSC Part # C25879 -> C4109
Connections:
- net +1V5: now also C132.1
- net GND: now also C132.2
Changed lines of the file:
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@@
 	(title_block
 		(title "Icepi CM0")
-		(date "2025-11-15")
+		(date "2025-11-21")
 		(rev "v1.0")
 		(company "Icy Electronics")
 		(comment 1 "Chengyin Yao (cheyao)")
 		(comment 2 "https://github.com/cheyao/icepi-cm0")
+		(comment 3 "License: Solderpad")
 	)
 	(bus_alias "ADDRESS"
@@
 	)
 	(junction
+		(at 243.84 152.4)
+		(diameter 0)
+		(color 0 0 0 0)
+	)
+	(junction
 		(at 177.8 118.11)
 		(diameter 0)
@@
 	)
 	(junction
+		(at 243.84 142.24)
+		(diameter 0)
+		(color 0 0 0 0)
+	)
+	(junction
 		(at 264.16 107.95)
 		(diameter 0)
@@
 		)
 	)
+	(wire
+		(pts
+			(xy 233.68 142.24) (xy 243.84 142.24)
+		)
+		(stroke
+			(width 0)
+			(type default)
+		)
+	)
 	(bus
 		(pts
@@
 	(wire
 		(pts
+			(xy 233.68 152.4) (xy 233.68 151.13)
+		)
+		(stroke
+			(width 0)
+			(type default)
+		)
+	)
+	(wire
+		(pts
 			(xy 71.12 109.22) (xy 77.47 109.22)
 		)
@@
 	(wire
 		(pts
+			(xy 243.84 152.4) (xy 233.68 152.4)
+		)
+		(stroke
+			(width 0)
+			(type default)
+		)
+	)
+	(wire
+		(pts
 			(xy 99.06 64.77) (xy 99.06 66.04)
 		)
@@
 	(wire
 		(pts
+			(xy 233.68 143.51) (xy 233.68 142.24)
+		)
+		(stroke
+			(width 0)
+			(type default)
+		)
+	)
+	(wire
+		(pts
 			(xy 213.36 116.84) (xy 213.36 118.11)
 		)
@@
 			)
 		)
-		(property "Value" "2.2k"
+		(property "Value" "2k"
 			(at 152.4 67.3099 0)
 			(effects
@@
 			)
 		)
-		(property "LCSC Part #" "C25879"
+		(property "LCSC Part #" "C4109"
 			(at 154.94 66.04 0)
 			(effects
@@
 	)
 	(symbol
+		(lib_id "Device:C")
+		(at 233.68 147.32 0)
+		(unit 1)
+		(exclude_from_sim no)
+		(in_bom yes)
+		(on_board yes)
+		(dnp no)
+		(property "Reference" "C132"
+			(at 234.442 144.78 0)
+			(effects
+				(font
+					(size 1.27 1.27)
+				)
+				(justify left)
+			)
+		)
+		(property "Value" "100nF"
+			(at 234.442 149.606 0)
+			(effects
+				(font
+					(size 1.27 1.27)
+				)
+				(justify left)
+			)
+		)
+		(property "Footprint" "Capacitor_SMD:C_0402_1005Metric"
+			(at 234.6452 151.13 0)
+			(effects
+				(font
+					(size 1.27 1.27)
+				)
+				(hide yes)
+			)
+		)
+		(property "Datasheet" "~"
+			(at 233.68 147.32 0)
+			(effects
+				(font
+					(size 1.27 1.27)
+				)
+				(hide yes)
+			)
+		)
+		(property "Description" "Unpolarized capacitor"
+			(at 233.68 147.32 0)
+			(effects
+				(font
+					(size 1.27 1.27)
+				)
+				(hide yes)
+			)
+		)
+		(property "LCSC Part #" "C1525"
+			(at 233.68 147.32 0)
+			(effects
+				(font
+					(size 1.27 1.27)
+				)
+				(hide yes)
+			)
+		)
+		(property "FT Position Offset" ""
+			(at 233.68 147.32 0)
+			(effects
+				(font
+					(size 1.27 1.27)
+				)
+				(hide yes)
+			)
+		)
+		(property "FT Rotation Offset" ""
+			(at 233.68 147.32 0)
+			(effects
+				(font
+					(size 1.27 1.27)
+				)
+				(hide yes)
+			)
+		)
+		(pin "2"
+		)
+		(pin "1"
+		)
+		(instances
+			(project "cm0"
+				(path "/b53f5dbb-8078-4818-9e8f-fdf90ba6d854/32a4bb18-2695-4537-bbd4-f872ec13cb53"
+					(reference "C132")
+					(unit 1)
+				)
+			)
+		)
+	)
+	(symbol
 		(lib_id "Device:R")
 		(at 154.94 76.2 0)
@@
 			)
 		)
-		(property "Value" "2.2k"
+		(property "Value" "2k"
 			(at 152.4 77.4699 0)
 			(effects
@@
 			)
 		)
-		(property "LCSC Part #" "C25879"
+		(property "LCSC Part #" "C4109"
 			(at 154.94 76.2 0)
 			(effects
