File: hardware/gpdi.kicad_sch (KiCad schematic)
At the start: 12 parts, among them J5 GPDI_A, Q3 BSN20, U19 UCL0524P, U20 UCL0524P, U23 UCL0524P

Commit message: Add fixes and improvements
Parts:
- R39, R40: value 2.2k -> 2k; LCSC Part # C25879 -> C4109
Changed lines of the file:
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@@
 	(title_block
 		(title "Icepi CM0")
-		(date "2025-11-15")
+		(date "2025-11-21")
 		(rev "v1.0")
 		(company "Icy Electronics")
 		(comment 1 "Chengyin Yao (cheyao)")
 		(comment 2 "https://github.com/cheyao/icepi-cm0")
+		(comment 3 "License: Solderpad")
 	)
 	(bus_alias "GPDI"
@@
 			)
 		)
-		(property "Value" "2.2k"
+		(property "Value" "2k"
 			(at 129.286 77.47 90)
 			(effects
@@
 			)
 		)
-		(property "LCSC Part #" "C25879"
+		(property "LCSC Part #" "C4109"
 			(at 127 77.47 0)
 			(effects
@@
 			)
 		)
-		(property "Value" "2.2k"
+		(property "Value" "2k"
 			(at 134.366 77.47 90)
 			(effects
@@
 			)
 		)
-		(property "LCSC Part #" "C25879"
+		(property "LCSC Part #" "C4109"
 			(at 132.08 77.47 0)
 			(effects
