File: hardware/power.kicad_sch (KiCad schematic)
At the start: 78 parts, among them Q1 BSN20, Q2 AO3415A, U3 SY8088, U4 SY8088, U5 SY8088, U6 SY8089A, U7 SY8113, U8 SY8088

Commit message: Add fixes and improvements
Parts:
- added C131: 100nF, Capacitor_SMD:C_0402_1005Metric, symbol Device:C
- R12, R15, R16, R25: value 10k -> 100k; LCSC Part # C25744 -> C25741
- R13, R17, R26: value 2.2k -> 22k; LCSC Part # C25879 -> C25768
- R14: value 15k -> 150k; LCSC Part # C25756 -> C2909320
Connections:
- net +3V3_IO: now also C131.2
- net +5V: now also C131.1
